File: macrokeyboard/bluetooth.kicad_sch (KiCad schematic)
At the start: 22 parts, among them J4 Conn_01x03, SW6 SW_Push, U2 nRF52810-QCxx, Y1 32.768KHz, Y2 32MHz

Commit message: PCB completion
Parts:
- removed NT1: NetTie_2, NetTie:NetTie-2_SMD_Pad0.5mm, symbol Device:NetTie_2
- added C41: 1.5pF, Capacitor_SMD:C_0402_1005Metric, symbol Device:C_Small
- added J7: Chip_ant, 1_macrokeys:KH5220-A36, symbol Connector:Conn_Coaxial_Small
- added L3: 4.3nH, Inductor_SMD:L_0402_1005Metric, symbol Device:L_Small
Connections:
- net ANT: now also C41.2, L3.1
- net GND: now also C41.1
- new net: J7.1 (In), L3.2
- no-connect marks 6 -> 7
