File: macrokeyboard/macrokeyboard.kicad_sch (KiCad schematic)
At the start: 36 parts

Commit message: important changes before order
Parts:
- removed D1, D10, D11, D12, D13, D14, D15, D16, D2, D5, D6, D7, D8, D9: 1N4148WS, Diode_SMD:D_SOD-323, symbol Diode:1N4148WS
- added D1, D10, D11, D12, D13, D14, D2, D3, D4, D5, D6, D7, D8, D9: 1N4148W, Diode_SMD:D_SOD-123, symbol Diode:1N4148W
Connections:
- net ROW1: now also D1.1 (K), D2.1 (K)
- net ROW2: now also D3.1 (K), D4.1 (K), D5.1 (K), D6.1 (K)
- net ROW3: now also D10.1 (K), D7.1 (K), D8.1 (K), D9.1 (K)
- net ROW4: now also D11.1 (K), D12.1 (K), D13.1 (K), D14.1 (K)
- net at S14.2: now also D12.2 (A)
- net at S7.2: now also D5.2 (A)
- net at S5.2: now also D3.2 (A)
- net at S12.2: now also D10.2 (A)
- net at S10.2: now also D8.2 (A)
- net at S6.2: now also D4.2 (A)
- net at S1.2: now also D1.2 (A)
- net at S13.2: now also D11.2 (A)
- net at S16.2: now also D14.2 (A)
- net at S2.2: now also D2.2 (A)
- net at S8.2: now also D6.2 (A)
- net at S11.2: now also D9.2 (A)
- net at S15.2: now also D13.2 (A)
- net at S9.2: now also D7.2 (A)
