File: macrokeyboard/MCU.kicad_sch (KiCad schematic)
At the start: 77 parts, among them J1 USB_C_Receptacle_USB2.0_16P, J2 Conn_01x02_MountingPin, J3 Conn_02x04_Odd_Even, J5 Conn_01x03, J6 Conn_01x02, Q1 Si1308EDL, SW1 SW_SPDT, SW2 SW_SPDT, SW3 SW_Push, SW4 SW_Push, SW5 SW_Push, U1 STM32F072VBTx, U3 BQ25186DLHR, U4 RV-3028-C7, U5 E-INK_Display_Conn, U6 TPS7A0233DBVR, U7 TPS7A0233DBVR

Commit message: important changes before order
Parts:
- removed SW1, SW2: SW_SPDT, 1_macrokeys:SK12D07VG4, symbol Switch:SW_SPDT
- added U8, U9: SK12D07VG4, 1_macrokeys:SK12D07VG4, symbol 1_macrokeys-lib:SK12D07VG4
Connections:
- net +3V3: now also U8.COM
- net GND: now also U9.1
- net PWR_EN: now also U9.COM
- net at R16.2: now also U9.2
- net at R20.1, U1.79 (PC11): now also U8.2
- net at R18.1, U1.78 (PC10): now also U8.1

Commit message: fabrication files
Parts:
- removed C34, C40: 1uF, Capacitor_SMD:C_0603_1608Metric, symbol Device:C_Small
- removed U7: TPS7A0233DBVR, 1_macrokeys:SOT_233DBVR_TEX, symbol 1_macrokeys-lib:TPS7A0233DBVR
- added R29: 10k, Resistor_SMD:R_0603_1608Metric, symbol Device:R_Small_US
- R19: value 1k -> 4.7k
- R24: value 1k -> 10k
- U6: value TPS7A0233DBVR -> DS8572-33S5
Connections:
- net +3V3: now also R24.2
- net GND: now also R29.1; no longer D24.1 (K)
- net at J6.1 (Pin_1), U4.6 (VBACKUP): now also R29.2
- net at U3.3 (*PG/GPO): now also D24.1 (K); no longer R24.2
Other:
- moved on the sheet: C11, C12, C13, D24, J2, R24, SW5, TH3, U3
